Commit message: Add modular method for sequential open loop control
Following changes:
- Add modular method in tail_controller.yaml ffor the sequential open loop control
- Increase tail torque limits
- Add plotjuggler_config_euler to have euler angles be graphed

File: quad_simulator/spirit_description/urdf/spirit_dira.urdf (robot description, URDF)
Before this commit: robot spirit, 20 links, 19 joints
Links:
- removed link tail_link_0
- removed link tail_link_1
- removed link tail_mass
Joints:
- removed joint body_tail_joint_0
- removed joint body_tail_joint_1
- removed joint tail_link_mass_joint

File: quad_simulator/spirit_description/urdf/spirit_gazebo_tail.urdf.xacro (robot description, xacro)
@@ -461,5 +461,5 @@
 		<axis xyz="1 0 0" />
 		<origin xyz="0 0 0" rpy="0 0 0" />
-		<limit effort="35" lower="-1.57" upper="1.57" velocity="1000000" />
+		<limit effort="50" lower="-1.57" upper="1.57" velocity="1000000" />
 		<dynamics damping="0.0" friction="0.0" />
 	</joint>
@@ -469,5 +469,5 @@
 		<axis xyz="0 1 0" />
 		<origin xyz="0 0 ${tailLength}" rpy="0 0 0" />
-		<limit effort="35" lower="-1.57" upper="1.57" velocity="1000000" />
+		<limit effort="50" lower="-1.57" upper="1.57" velocity="1000000" />
 		<dynamics damping="0.0" friction="0.0" />
 	</joint>
