Commit message: Add working ICRA run
Following were changed:
- Add python script to run multiple ICRA world
- Integrated global_body_planner.yaml to be ran when running quad_plan.launch (this lets you reset goal, etc.)
- Add different configuration to global_body_planner, spirit, and local_planner yaml files (e.g. different planning params, gait phases, etc.)
- Fixed unwrapping yaw ref issue

File: quad_simulator/spirit_description/urdf/spirit.urdf (robot description, URDF)
Before this commit: robot spirit, 20 links, 19 joints
Links:
- removed link text_left
- removed link text_right
Joints:
- removed joint cmu_text_left
- removed joint cmu_text_right
