Commit message: Update s.t. can load ICRA world
Some parameter tuning & commnets:
- Increase toe of spirit
- Change location of goal and start
- Decrease nominal sampling speed

File: quad_simulator/a1_description/xacro/const.xacro (robot description, xacro)
@@ -16,5 +16,5 @@
     <xacro:property name="calf_width" value="0.016"/>
     <xacro:property name="calf_height" value="0.016"/>
-    <xacro:property name="foot_radius" value="0.02"/>
+    <xacro:property name="foot_radius" value="0.03"/> <!-- Original: 0.02-->
     <xacro:property name="stick_radius" value="0.01"/>
     <xacro:property name="stick_length" value="0.2"/>

File: quad_simulator/a1_description/xacro/leg.xacro (robot description, xacro)
@@ -129,5 +129,5 @@
                     <sphere radius="${foot_radius-0.01}"/>
                 </geometry>
-                <material name="orange"/>
+                <material name="white"/>
             </visual>
             <collision name="toe${suffix}_collision">

File: quad_simulator/spirit_description/urdf/spirit.urdf (robot description, URDF)
Before this commit: robot spirit, 20 links, 19 joints
Links:
- link toe0: geometry collision sphere radius=0.03; visual sphere radius=0.03
- link toe1: geometry collision sphere radius=0.03; visual sphere radius=0.03
- link toe2: geometry collision sphere radius=0.03; visual sphere radius=0.03
- link toe3: geometry collision sphere radius=0.03; visual sphere radius=0.03

File: quad_simulator/spirit_description/urdf/spirit_meshes.urdf (robot description, URDF)
Before this commit: robot spirit, 18 links, 17 joints
Links:
- link toe0: geometry collision sphere radius=0.05; visual sphere radius=0.05
- link toe1: geometry collision sphere radius=0.05; visual sphere radius=0.05
- link toe2: geometry collision sphere radius=0.05; visual sphere radius=0.05
- link toe3: geometry collision sphere radius=0.05; visual sphere radius=0.05
